File: Motor-interface.kicad_pcb (KiCad board)
At the start: 2 copper layers, 20 parts, among them J1 RJ45, K1 RELAY_2RT, P1 CONN_01X02, P2 TE-23pins connector, Q1 Q_NPN_BCE, U1 MCP42010, U2 Teensy_3.2, U3 TLP2361, U4 TLP2361, U5 MCP2551-I/SN

Commit message: most associations, started pcb
Parts:
- removed C1: 4.7nF, Capacitors_SMD:C_1206
- removed D1: PESD1CAN, TO_SOT_Packages_SMD:SOT-23_Handsoldering
- removed J1: RJ45, Connect:RJ45_8
- removed JP1, JP2: Terminate, electric_car_lib:JumperSingle
- removed JP3: Filter, electric_car_lib:JumperSingle
- removed K1: RELAY_2RT, Relays_ThroughHole:Relay_SANYOU_SRD_Series_Form_C
- removed P1: CONN_01X02, Connect:bornier2
- removed P2: TE-23pins connector, electric_car_lib:TE_23_pins_776087-1_connector
- removed Q1: Q_NPN_BCE, TO_SOT_Packages_SMD:SOT-23
- removed R1: 100, Resistors_SMD:R_1210_HandSoldering
- removed R2: 330, Resistors_SMD:R_1210_HandSoldering
- removed R3: 4.7K, Resistors_SMD:R_1210_HandSoldering
- removed R4, R5: 60, Resistors_SMD:R_1210_HandSoldering
- removed U1: MCP42010, Housings_SOIC:SOIC-14_3.9x8.7mm_Pitch1.27mm
- removed U2: Teensy_3.2, Housings_SSOP:TSSOP-32_6.1x11mm_Pitch0.65mm
- removed U3, U4: TLP2361, electric_car_lib:soic-5
- removed U5: MCP2551-I/SN, Power_Integrations:SO-8
- added C101: C, Capacitors_SMD:C_1210_HandSoldering, F.Cu at (120.7, 135.9)
- added C201: 4.7nF, Capacitors_SMD:C_1210_HandSoldering, F.Cu at (227.3, 49.5)
- added D101: D, Diodes_SMD:DO-214AB_Handsoldering, F.Cu at (33.0, 90.2)
- added D201: PESD1CAN, TO_SOT_Packages_SMD:SOT-23_Handsoldering, F.Cu at (45.7, -3.81)
- added J101: 0, Resistors_SMD:R_1210_HandSoldering, F.Cu at (-33.0, 14.0)
- added J102: 0, Resistors_SMD:R_1210_HandSoldering, F.Cu at (29.2, -7.62)
- added J201: RJ45, Connect:RJ45_8, F.Cu at (116.8, 35.6)
- added J202: RJ45, Connect:RJ45_8, F.Cu at (144.8, 30.5)
- added JP201: Terminate, electric_car_lib:JumperSingle, F.Cu at (-48.3, -5.08)
- added JP202: Terminate, electric_car_lib:JumperSingle, F.Cu at (-21.6, 19.1)
- added JP203: Filter, electric_car_lib:JumperSingle, F.Cu at (-22.9, 0.00)
- added K101: RELAY_2RT, Relays_ThroughHole:Relay_SANYOU_SRD_Series_Form_C, F.Cu at (203.2, 21.6)
- added P101: TE-23pins connector, electric_car_lib:TE_23_pins_776087-1_connector, F.Cu at (127.0, 168.9)
- added P102: PSU_ISO, Pin_Headers:Pin_Header_Straight_1x04, F.Cu at (266.7, 68.6)
- added P103: Halls, Pin_Headers:Pin_Header_Straight_1x06, F.Cu at (167.6, 161.3)
- added P104: LineContactor, Connect:bornier2, F.Cu at (45.7, 127.0)
- added P105: ReverseContactor, Connect:bornier2, F.Cu at (44.5, 119.4)
- added P106: FanContactor, Connect:bornier2, F.Cu at (53.3, 153.7)
- added P108: MC_USB, Pin_Headers:Pin_Header_Straight_1x04, F.Cu at (78.7, 168.9)
- added P109: MC_CAN, Pin_Headers:Pin_Header_Straight_1x04, F.Cu at (87.6, 170.2)
- added Q101: Q_NPN_BCE, TO_SOT_Packages_SMD:SOT-23, F.Cu at (36.8, 6.35)
- added R101: 10k, Resistors_SMD:R_1206_HandSoldering, F.Cu at (-34.3, -29.2)
- added R102: 10k, Resistors_SMD:R_1206_HandSoldering, F.Cu at (22.9, -1.27)
- added R103: 10k, Resistors_SMD:R_1206_HandSoldering, F.Cu at (20.3, -10.2)
- added R104: 1k, Resistors_SMD:R_1206_HandSoldering, F.Cu at (14.0, 8.89)
- added R105: 1k, Resistors_SMD:R_1206_HandSoldering, F.Cu at (0.00, 33.0)
- added R106: 1k, Resistors_SMD:R_1206_HandSoldering, F.Cu at (-8.89, 31.8)
- added R107: 100, Resistors_SMD:R_1206_HandSoldering, F.Cu at (16.5, 40.6)
- added R108: 100, Resistors_SMD:R_1206_HandSoldering, F.Cu at (-5.08, 20.3)
- added R109: 100, Resistors_SMD:R_1206_HandSoldering, F.Cu at (19.1, 29.2)
- added R110: 100, Resistors_SMD:R_1206_HandSoldering, F.Cu at (-17.8, 3.81)
- added R111: 100, Resistors_SMD:R_1206_HandSoldering, F.Cu at (33.0, 15.2)
- added R112: 100, Resistors_SMD:R_1206_HandSoldering, F.Cu at (12.7, 24.1)
- added R113: 1k, Resistors_SMD:R_1206_HandSoldering, F.Cu at (-27.9, -8.89)
- added R114: 1k, Resistors_SMD:R_1206_HandSoldering, F.Cu at (6.35, -15.2)
- added R115: 100, Resistors_SMD:R_1206_HandSoldering, F.Cu at (-7.62, -5.08)
- added R201: 100, Resistors_SMD:R_1206_HandSoldering, F.Cu at (10.2, -5.08)
- added R202: 330, Resistors_SMD:R_1206_HandSoldering, F.Cu at (-5.08, 7.62)
- added R203: 4.7K, Resistors_SMD:R_1206_HandSoldering, F.Cu at (31.8, 7.62)
- added R204: 60, Resistors_SMD:R_1210_HandSoldering, F.Cu at (39.4, -16.5)
- added R205: 60, Resistors_SMD:R_1210_HandSoldering, F.Cu at (-61.0, 55.9)
- added R301: 1k, Resistors_SMD:R_1206_HandSoldering, F.Cu at (44.5, 22.9)
- added R302: 1k, Resistors_SMD:R_1206_HandSoldering, F.Cu at (29.2, 30.5)
- added R303: 1k, Resistors_SMD:R_1206_HandSoldering, F.Cu at (83.8, 69.8)
- added R304: 1k, Resistors_SMD:R_1206_HandSoldering, F.Cu at (114.3, 71.1)
- added R305: 1k, Resistors_SMD:R_1206_HandSoldering, F.Cu at (57.1, 47.0)
- added R306: 1k, Resistors_SMD:R_1206_HandSoldering, F.Cu at (41.9, 73.7)
- added R307: 1k, Resistors_SMD:R_1206_HandSoldering, F.Cu at (-3.81, 53.3)
- added R308: 1k, Resistors_SMD:R_1206_HandSoldering, F.Cu at (25.4, 58.4)
- added U101: AP1117D50, TO_SOT_Packages_SMD:TO-252-2Lead, F.Cu at (268.0, 54.6)
- added U102: AP1117D33, TO_SOT_Packages_SMD:TO-252-2Lead, F.Cu at (299.7, 77.5)
- added U103: TLP2361, electric_car_lib:soic-5, F.Cu at (-34.3, -10.2)
- added U104: TLP2361, electric_car_lib:soic-5, F.Cu at (8.89, -22.9)
- added U105: TLP2361, electric_car_lib:soic-5, F.Cu at (35.6, 24.1)
- added U106: TLP2361, electric_car_lib:soic-5, F.Cu at (57.1, 11.4)
- added U107: TLP2361, electric_car_lib:soic-5, F.Cu at (87.6, 91.4)
- added U108: TLP2361, electric_car_lib:soic-5, F.Cu at (7.62, 64.8)
- added U109: Teensy_3.2, Housings_SSOP:TSSOP-32_6.1x11mm_Pitch0.65mm, F.Cu at (-8.89, -20.3)
- added U110: TLP2361, electric_car_lib:soic-5, F.Cu at (-20.3, 33.0)
- added U201: TLP2361, electric_car_lib:soic-5, F.Cu at (-33.0, 45.7)
- added U202: TLP2361, electric_car_lib:soic-5, F.Cu at (-74.9, 35.6)
- added U203: MCP2551-I/SN, Power_Integrations:SO-8, F.Cu at (-39.4, 0.00)
- added U301: MCP42010, Housings_SOIC:SOIC-14_3.9x8.7mm_Pitch1.27mm, F.Cu at (21.6, -24.1)
- added U302: TLP2361, electric_car_lib:soic-5, F.Cu at (-47.0, 77.5)
- added U303: TLP2361, electric_car_lib:soic-5, F.Cu at (-3.81, 120.7)
- added U304: TLP2361, electric_car_lib:soic-5, F.Cu at (113.0, -21.6)
- added U305: TLP2361, electric_car_lib:soic-5, F.Cu at (96.5, 1.27)

Commit message: removed files from other repo
Parts:
- moved U102 246.3 mm to (58.4, 127.0)
- moved R101 215.8 mm to (62.2, 163.8)
- moved P102 198.0 mm to (77.5, 127.0), turned to 180 degrees
- moved R104 195.8 mm to (90.2, 189.2)
- moved U302 186.2 mm to (113.0, 172.7), turned to 270 degrees
- moved U103 185.7 mm to (48.3, 156.2)
- moved R114 185.5 mm to (54.6, 163.8)
- moved R106 182.1 mm to (82.5, 189.2)
- moved U202 171.0 mm to (59.7, 141.0), turned to 180 degrees
- moved R105 171.0 mm to (77.5, 185.4), turned to 270 degrees
- moved JP201 170.8 mm to (38.1, 142.2)
- moved U109 167.2 mm to (95.2, 110.5)
- moved U203 165.7 mm to (45.7, 142.2), turned to 90 degrees
- moved JP203 164.1 mm to (38.1, 152.4)
- moved R204 161.5 mm to (31.8, 144.8), turned to 90 degrees
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Routing:
- net /Contactor+Common: track 0.00 -> 78.5 mm, vias 0 -> 11
- net GND: track 0.00 -> 62.5 mm, vias 0 -> 3
- net /Line-contactor-coil: track 0.00 -> 49.7 mm, vias 0 -> 4
- net /Fan-contactor-coil: track 0.00 -> 39.6 mm, vias 0 -> 2
- net /Motor_CAN-L: track 0.00 -> 34.7 mm
- net /USB-Programmer-Wires-TX: track 0.00 -> 31.3 mm, vias 0 -> 2
- net /PotsSwitches/Motor_5V: track 0.00 -> 25.5 mm, vias 0 -> 4
- net /Motor_CAN-H: track 0.00 -> 23.6 mm, vias 0 -> 4
- net Net-(R101-Pad1): track 0.00 -> 20.4 mm
- net Net-(JP203-Pad1): track 0.00 -> 19.5 mm
- net /Motor-temperature: track 0.00 -> 11.3 mm
- net /Hall_GND: track 0.00 -> 10.7 mm
- net /Hall_Power: track 0.00 -> 10.1 mm
- net Net-(JP202-Pad2): track 0.00 -> 9.96 mm
- net /Motor-sensor-C: track 0.00 -> 9.53 mm
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
Commit message: PBC layout
Parts:
- U109: footprint Housings_SSOP:TSSOP-32_6.1x11mm_Pitch0.65mm -> electric_car_lib:Teensy3.2_inv
- moved U302 163.7 mm to (181.6, 24.1), turned to 90 degrees
- moved C201 163.6 mm to (87.6, 134.6)
- moved R113 160.1 mm to (156.2, 152.4)
- moved R302 157.4 mm to (176.5, 34.3)
- moved U303 157.3 mm to (160.0, 29.2)
- moved U106 151.8 mm to (85.1, 167.6), turned to 270 degrees
- moved U108 151.6 mm to (85.1, 172.7), turned to 270 degrees
- moved R110 149.8 mm to (101.6, 166.4), turned to 180 degrees
- moved R112 148.9 mm to (99.1, 171.4), turned to 270 degrees
- moved U101 145.9 mm to (128.3, 96.5)
- moved R114 138.5 mm to (190.5, 137.2)
- moved R111 136.5 mm to (101.6, 163.8), turned to 180 degrees
- moved U110 131.7 mm to (184.2, 141.0)
- moved R115 126.3 mm to (184.2, 130.8)
- moved R108 118.1 mm to (50.8, 124.5)
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Routing:
- net GND: track 62.5 -> 554.9 mm, vias 3 -> 26
- net /PotsSwitches/Motor_5V: track 25.5 -> 471.7 mm, vias 4 -> 24
- net +3V3: track 0.00 -> 427.7 mm, vias 0 -> 23
- net /PotsSwitches/BrakePot: track 0.00 -> 270.8 mm, vias 0 -> 14
- net /PotsSwitches/AccelPot: track 0.00 -> 256.7 mm, vias 0 -> 22
- net GNDA: track 0.00 -> 192.8 mm, vias 0 -> 8
- net /PotsSwitches/DP-CS: track 0.00 -> 158.3 mm, vias 0 -> 8
- net /Motor_Logic_On: track 0.00 -> 143.0 mm
- net /MOT_ON: track 0.00 -> 137.7 mm
- net +12V: track 0.00 -> 115.5 mm, vias 0 -> 5
- net /CANmodule/CAN_TX: track 0.00 -> 107.8 mm, vias 0 -> 2
- net /CANmodule/CAN_RX: track 0.00 -> 103.3 mm, vias 0 -> 2
- net /PotsSwitches/MISO: track 0.00 -> 99.0 mm, vias 0 -> 7
- net Net-(R101-Pad1): track 20.4 -> 118.5 mm
- net /Contactor+Common: track 78.5 -> 171.8 mm, vias 11 -> 6
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
Commit message: minor tweaks, started layout
Parts:
- removed D101: D, Diodes_SMD:DO-214AB_Handsoldering
- removed K101: RELAY_2RT, Relays_ThroughHole:Relay_SANYOU_SRD_Series_Form_C
- added P107: Battery+, Connect:bornier2, F.Cu at (154.9, 146.1)
- added R206: 100, Resistors_SMD:R_1206_HandSoldering, F.Cu at (56.5, 40.0)
- added U111: FODM3052, electric_car_lib:MFP4L, F.Cu at (141.0, 144.8)
- added U306: TLP290-4, SMD_Packages:SO-16-N, F.Cu at (24.1, 168.9)
- C101: value C -> 10uF
- Q101: footprint TO_SOT_Packages_SMD:SOT-23 -> TO_SOT_Packages_SMD:SOT-428
- U101, U102: footprint TO_SOT_Packages_SMD:TO-252-2Lead -> TO_SOT_Packages_SMD:SOT-223
- U301: value MCP42010 -> MCP4251; footprint Housings_SOIC:SOIC-14_3.9x8.7mm_Pitch1.27mm -> SMD_Packages:SOIC-14_N
- moved R305 134.8 mm to (31.8, 152.4)
- moved C101 134.7 mm to (73.7, 147.3)
- moved R301 134.7 mm to (82.5, 133.3)
- moved R302 134.7 mm to (92.7, 139.7)
- moved R303 134.7 mm to (74.9, 154.9)
- moved R304 134.7 mm to (104.1, 121.9)
- moved U301 134.7 mm to (74.9, 123.2)
- moved U302 134.7 mm to (97.8, 129.5)
- moved U303 134.7 mm to (76.2, 134.6)
- moved U304 134.7 mm to (83.8, 143.5)
- moved U305 134.7 mm to (92.7, 121.9)
- moved R308 131.2 mm to (29.2, 158.8)
- moved R306 131.1 mm to (19.1, 152.4)
- moved R307 127.0 mm to (20.3, 160.0)
- moved C201 104.0 mm to (44.5, 40.0), turned to 90 degrees
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Connections:
- C201 pad 1: GNDA -> Net-(C201-Pad1)
- JP203 pad 1: Net-(JP203-Pad1) -> Net-(C201-Pad1)
- JP203 pad 2: Net-(C201-Pad2) -> GNDA
- Q101 pad 3: GND -> /On/Off-Switch
- R113 pad 1: Net-(Q101-Pad1) -> Net-(R113-Pad1)
- R204 pad 1: Net-(JP203-Pad1) -> Net-(C201-Pad2)
- R205 pad 1: Net-(JP203-Pad1) -> Net-(C201-Pad2)
- U201 pad 5: /CANmodule/CAN_RX -> Net-(R206-Pad2)
Routing:
- net GND: track 554.9 -> 0.00 mm, vias 26 -> 0
- net /PotsSwitches/Motor_5V: track 471.7 -> 0.00 mm, vias 24 -> 0
- net +3V3: track 427.7 -> 0.00 mm, vias 23 -> 0
- net /PotsSwitches/BrakePot: track 270.8 -> 0.00 mm, vias 14 -> 0
- net /PotsSwitches/AccelPot: track 256.7 -> 0.00 mm, vias 22 -> 0
- net GNDA: track 192.8 -> 0.00 mm, vias 8 -> 0
- net /Contactor+Common: track 171.8 -> 0.00 mm, vias 6 -> 0
- net /PotsSwitches/DP-CS: track 158.3 -> 0.00 mm, vias 8 -> 0
- net /Motor_Logic_On: track 143.0 -> 0.00 mm
- net /MOT_ON: track 137.7 -> 0.00 mm
- net Net-(R101-Pad1): track 118.5 -> 0.00 mm
- net +12V: track 115.5 -> 0.00 mm, vias 5 -> 0
- net /CANmodule/CAN_TX: track 107.8 -> 0.00 mm, vias 2 -> 0
- net /CANmodule/CAN_RX: track 103.3 -> 0.00 mm, vias 2 -> 0
- net /PotsSwitches/MISO: track 99.0 -> 0.00 mm, vias 7 -> 0
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